Commit message: replacing urdf by xacro

File: src/alice_description/urdf/alice_description.urdf (robot description, URDF)
Before this commit: robot alice_description, 63 links, 62 joints
Joints:
- removed joint r_r_up_bottom_actuator_lig_joint
- added joint r_l_up_bottom_actuator_lig_joint: type continuous, parent r_l_up_leg_atuador, child r_l_up_bottom_actuator_lig, origin xyz=0.01969 -0.01016 -0.01972 rpy=2.89563081079793 1.5707963267949 0, axis 1 0 0
- joint l_back_up_leg_bar_joint: axis 0 0.999717465199625 -0.0237695135590915 -> 0 1 0; origin xyz=-0.0147907980872848 0.0168343365597003 0.0496138736547796 rpy=3.14137187381274 0.135752874403086 -0.00324767223227192 -> xyz=-0.1447908 0.0168343365597003 0.04998587 rpy=3.14137187381274 0.135752874403086 -0.00324767223227192
- joint l_l_up_bottom_actuator_lig_joint: axis 0 0 0 -> 1 0 0; origin xyz=0.0308556196868716 -0.0189473349665785 -0.0221220000000291 rpy=-1.04104620894622 1.57079630098533 2.3190651342933 -> xyz=0.01969 -0.01016 -0.0221220000000291 rpy=-1.04104620894622 1.57079630098533 2.3190651342933; type fixed -> continuous
- joint l_r_up_bottom_actuator_lig_joint: axis 0 0 0 -> 1 0 0; origin xyz=0.0309326457985631 -0.0188485248454831 -0.0196480000000081 rpy=2.91425644849924 1.5707963267949 0 -> xyz=0.01969 -0.01016 -0.0196480000000081 rpy=2.91425644849924 1.5707963267949 0; type fixed -> continuous
- joint r_back_up_leg_bar_r_leg_middle_joint: axis 0 0 0 -> 0 1 0; origin xyz=0.033308707160086 -0.0285840269311472 -0.654109777039992 rpy=-5.88705488029949E-05 0.0702982984060446 -0.0016741881463759 -> xyz=0.04044594 0.00622512 -0.26182126 rpy=-5.88705488029949E-05 0.0702982984060446 -0.0016741881463759; type fixed -> continuous
- joint r_r_up_leg_atuador_r_r_up_bottom_actuator_lig_joint: axis 0 0 0 -> 1 0 0; origin xyz=0.031177 -0.018522 -0.019648 rpy=2.8454 1.5708 -0.040242 -> xyz=0.01969 -0.01016 -0.019648 rpy=2.8454 1.5708 -0.040242; type fixed -> continuous
