Commit message: update

File: src/alice_xacro_desc/urdf/robot.urdf.xacro (robot description, xacro)
@@ -7,4 +7,6 @@
   <xacro:include filename="up_act_segment.xacro" />
   <xacro:include filename="center_leg.xacro" />
+  <xacro:include filename="arms.xacro" />
+  <xacro:include filename="head.xacro" />
   <link name="base_footprint"/>
   <joint name="base_footprint_joint" type="fixed">
@@ -27,4 +29,16 @@
     </inertial>
   </link>
+  <!-- Instanciando o Braço Esquerdo -->
+  <xacro:head parent="base_link">
+    <origin xyz="0.05513968 -0.00242679 0.246" rpy="0 0 0" />
+  </xacro:head>
+  <!-- Instanciando o Braço Esquerdo -->
+  <xacro:left_arm parent="base_link">
+    <origin xyz="0.03325 0.222 0.152" rpy="0 0 0" />
+  </xacro:left_arm>
+  <!-- Instanciando o Braço Direito -->
+  <xacro:right_arm parent="base_link">
+    <origin xyz="0.03325 -0.222 0.152" rpy="0 0 0" />
+  </xacro:right_arm>
   <!-- Instanciando a Perna Esquerda -->
   <xacro:up_actuator_segment prefix="l_l" parent="base_link">

Commit message: adds display.rviz file

File: src/alice_xacro_desc/urdf/robot.urdf.xacro (robot description, xacro)
@@ -13,5 +13,5 @@
     <parent link="base_footprint"/>
     <child link="base_link"/>
-    <origin xyz="0 0 0.7" rpy="0 0 0" />
+    <origin xyz="0 0 1.0" rpy="0 0 0" />
   </joint>
   <!-- Base do Robô -->

File: src/install/alice_xacro_desc/share/alice_xacro_desc/urdf/robot.urdf.xacro (robot description, xacro)
@@ -6,4 +6,7 @@
   <xacro:include filename="head.xacro" /> -->
   <xacro:include filename="up_act_segment.xacro" />
+  <xacro:include filename="center_leg.xacro" />
+  <xacro:include filename="arms.xacro" />
+  <xacro:include filename="head.xacro" />
   <link name="base_footprint"/>
   <joint name="base_footprint_joint" type="fixed">
@@ -26,12 +29,36 @@
     </inertial>
   </link>
+  <!-- Instanciando o Braço Esquerdo -->
+  <xacro:head parent="base_link">
+    <origin xyz="0.05513968 -0.00242679 0.246" rpy="0 0 0" />
+  </xacro:head>
+  <!-- Instanciando o Braço Esquerdo -->
+  <xacro:left_arm parent="base_link">
+    <origin xyz="0.03325 0.222 0.152" rpy="0 0 0" />
+  </xacro:left_arm>
+  <!-- Instanciando o Braço Direito -->
+  <xacro:right_arm parent="base_link">
+    <origin xyz="0.03325 -0.222 0.152" rpy="0 0 0" />
+  </xacro:right_arm>
   <!-- Instanciando a Perna Esquerda -->
   <xacro:up_actuator_segment prefix="l_l" parent="base_link">
-    <origin xyz="0 -0.15 -0.25" rpy="0 0 0" />
+    <origin xyz="-0.085 0.1685 -0.245" rpy="0 0 0" />
+  </xacro:up_actuator_segment>
+  <xacro:center_leg prefix="l" parent="base_link">
+    <origin xyz="-0.032 0.1075 -0.2365" rpy="0 0 0" />
+  </xacro:center_leg>
+  <xacro:up_actuator_segment prefix="l_r" parent="base_link">
+    <origin xyz="-0.085 0.0485 -0.245" rpy="0 0 0" />
   </xacro:up_actuator_segment>
   <!-- Instanciando a Perna Esquerda -->
-  <!-- <xacro:up_actuator_segment prefix="left" parent="base_link">
-    <origin xyz="0 0.15 -0.25" rpy="0 0 0" />
-  </xacro:biped_leg> -->
+  <xacro:up_actuator_segment prefix="r_l" parent="base_link">
+    <origin xyz="-0.085 -0.0485 -0.245" rpy="0 0 0" />
+  </xacro:up_actuator_segment>
+  <xacro:center_leg prefix="r" parent="base_link">
+    <origin xyz="-0.032 -0.1075 -0.2365" rpy="0 0 0" />
+  </xacro:center_leg>
+  <xacro:up_actuator_segment prefix="r_r" parent="base_link">
+    <origin xyz="-0.085 -0.1685 -0.245" rpy="0 0 0" />
+  </xacro:up_actuator_segment>
   <!-- O mesmo padrão se aplica para braços e cabeça -->
 </robot>

File: src/install/alice_xacro_desc/share/alice_xacro_desc/urdf/up_act_segment.xacro (robot description, xacro)
@@ -41,5 +41,5 @@
       type="continuous">
       <origin
-        xyz="0 0 0"
+        xyz="0 0 -0.025"
         rpy="0 0 0" />
       <parent
@@ -50,4 +50,61 @@
         xyz="0 1 0" />
     </joint>
+    <link name="${prefix}_up_atuador">
+      <visual>
+        <geometry>
+          <!-- Reutilizando o mesmo STL -->
+          <mesh filename="package://alice_xacro_desc/meshes/up_actuator.stl" />
+        </geometry>
+      </visual>
+      <inertial>
+        <mass value="1.0" />
+        <origin xyz="0 0 0" rpy="0 0 0" />
+        <inertia ixx="0.01" ixy="0.0" ixz="0.0" iyy="0.01" iyz="0.0" izz="0.01" />
+      </inertial>
+    </link>
+    <joint
+      name="${prefix}_up_haste_${prefix}_up_atuador_joint"
+      type="prismatic">
+      <origin
+        xyz="0 0 -0.075"
+        rpy="0 0 0" />
+      <parent
+        link="${prefix}_up_haste" />
+      <child
+        link="${prefix}_up_atuador" />
+      <axis
+        xyz="0 0 1" />
+      <limit
+        lower="-0.2"
+        upper="0.2"
+        effort="100"
+        velocity="1" />
+    </joint>
+    <link name="${prefix}_up_dn_leg_conn">
+      <visual>
+        <geometry>
+          <!-- Reutilizando o mesmo STL -->
+          <mesh filename="package://alice_xacro_desc/meshes/up_actuator_lig.stl" />
+        </geometry>
+      </visual>
+      <inertial>
+        <mass value="1.0" />
+        <origin xyz="0 0 0" rpy="0 0 0" />
+        <inertia ixx="0.01" ixy="0.0" ixz="0.0" iyy="0.01" iyz="0.0" izz="0.01" />
+      </inertial>
+    </link>
+    <joint
+      name="${prefix}_up_atuador_${prefix}_up_dn_leg_conn_joint"
+      type="continuous">
+      <origin
+        xyz="-0.001651 0 -0.1700170"
+        rpy="0 0 0" />
+      <parent
+        link="${prefix}_up_atuador" />
+      <child
+        link="${prefix}_up_dn_leg_conn" />
+      <axis
+        xyz="0 1 0" />
+    </joint>
     <!-- Aqui você continuaria declarando as juntas (ex: prismática para o atuador) e links (haste, conector final) usando sempre ${prefix}_nome_do_link -->
   </xacro:macro>
