Commit message: fixed CoM for URDF

File: src/alice_xacro_desc/urdf/arms.xacro (robot description, xacro)
@@ -18,7 +18,13 @@
       </visual>
       <inertial>
-        <mass value="1.0" />
-        <origin xyz="0 0 0" rpy="0 0 0" />
-        <inertia ixx="0.01" ixy="0.0" ixz="0.0" iyy="0.01" iyz="0.0" izz="0.01" />
+        <origin xyz="0.00280 0.01782 -0.06268" rpy="0 0 0"/>
+        <mass value="0.25180"/>
+        <inertia
+            ixx="0.003326125"
+            ixy="0.000001544"
+            ixz="0.000075089"
+            iyy="0.003336491"
+            iyz="-0.000034114"
+            izz="0.000059530"/>
       </inertial>
     </link>
@@ -31,7 +37,13 @@
       </visual>
       <inertial>
-        <mass value="1.0" />
-        <origin xyz="0 0 0" rpy="0 0 0" />
-        <inertia ixx="0.01" ixy="0.0" ixz="0.0" iyy="0.01" iyz="0.0" izz="0.01" />
+        <origin xyz="0.0 0.0 -0.05194" rpy="0 0 0"/>
+        <mass value="0.29579"/>
+        <inertia
+            ixx="0.000366379"
+            ixy="0.0"
+            ixz="0.0"
+            iyy="0.000366533"
+            iyz="0.0"
+            izz="0.000014856"/>
       </inertial>
     </link>
@@ -57,7 +69,13 @@
       </visual>
       <inertial>
-        <mass value="1.0" />
-        <origin xyz="0 0 0" rpy="0 0 0" />
-        <inertia ixx="0.01" ixy="0.0" ixz="0.0" iyy="0.01" iyz="0.0" izz="0.01" />
+        <origin xyz="-0.01764 -0.00010 -0.09055" rpy="0 0 0"/>
+        <mass value="0.34367"/>
+        <inertia
+            ixx="0.000927312"
+            ixy="0.000000789"
+            ixz="0.000065314"
+            iyy="0.001049676"
+            iyz="0.000001769"
+            izz="0.000190178"/>
       </inertial>
     </link>
@@ -88,7 +106,13 @@
       </visual>
       <inertial>
-        <mass value="1.0" />
-        <origin xyz="0 0 0" rpy="0 0 0" />
-        <inertia ixx="0.01" ixy="0.0" ixz="0.0" iyy="0.01" iyz="0.0" izz="0.01" />
+        <origin xyz="0.11743 0.00195 0.00186" rpy="0 0 0"/>
+        <mass value="0.34308"/>
+        <inertia
+            ixx="0.000076037"
+            ixy="0.000113102"
+            ixz="-0.000034335"
+            iyy="0.003507890"
+            iyz="-0.000002022"
+            izz="0.003475583"/>
       </inertial>
     </link>
@@ -124,7 +148,13 @@
       </visual>
       <inertial>
-        <mass value="1.0" />
-        <origin xyz="0 0 0" rpy="0 0 0" />
-        <inertia ixx="0.01" ixy="0.0" ixz="0.0" iyy="0.01" iyz="0.0" izz="0.01" />
+        <origin xyz="0.00307 -0.01783 -0.06332" rpy="0 0 0"/>
+        <mass value="0.25180"/>
+        <inertia
+            ixx="0.003330078"
+            ixy="-0.000001676"
+            ixz="0.000081997"
+            iyy="0.003341524"
+            iyz="0.000035021"
+            izz="0.000060631"/>
       </inertial>
     </link>
@@ -137,7 +167,13 @@
       </visual>
       <inertial>
-        <mass value="1.0" />
-        <origin xyz="0 0 0" rpy="0 0 0" />
-        <inertia ixx="0.01" ixy="0.0" ixz="0.0" iyy="0.01" iyz="0.0" izz="0.01" />
+        <origin xyz="0.0 0.0 -0.05194" rpy="0 0 0"/>
+        <mass value="0.29579"/>
+        <inertia
+            ixx="0.000366379"
+            ixy="0.0"
+            ixz="0.0"
+            iyy="0.000366533"
+            iyz="0.0"
+            izz="0.000014856"/>
       </inertial>
     </link>
@@ -163,7 +199,13 @@
       </visual>
       <inertial>
-        <mass value="1.0" />
-        <origin xyz="0 0 0" rpy="0 0 0" />
-        <inertia ixx="0.01" ixy="0.0" ixz="0.0" iyy="0.01" iyz="0.0" izz="0.01" />
+        <origin xyz="-0.01764 -0.00010 -0.09055" rpy="0 0 0"/>
+        <mass value="0.34367"/>
+        <inertia
+            ixx="0.000927312"
+            ixy="0.000000789"
+            ixz="0.000065314"
+            iyy="0.001049676"
+            iyz="0.000001769"
+            izz="0.000190178"/>
       </inertial>
     </link>
@@ -194,7 +236,13 @@
       </visual>
       <inertial>
-        <mass value="1.0" />
-        <origin xyz="0 0 0" rpy="0 0 0" />
-        <inertia ixx="0.01" ixy="0.0" ixz="0.0" iyy="0.01" iyz="0.0" izz="0.01" />
+        <origin xyz="0.16920 -0.00421 0.00107" rpy="0 0 0"/>
+        <mass value="0.05993"/>
+        <inertia
+            ixx="0.000017279"
+            ixy="-0.000028339"
+            ixz="-0.000011329"
+            iyy="0.000716453"
+            iyz="0.000000559"
+            izz="0.000707547"/>
       </inertial>
     </link>

File: src/alice_xacro_desc/urdf/center_leg.xacro (robot description, xacro)
@@ -19,7 +19,13 @@
       </visual>
       <inertial>
-        <mass value="1.0" />
-        <origin xyz="0 0 0" rpy="0 0 0" />
-        <inertia ixx="0.01" ixy="0.0" ixz="0.0" iyy="0.01" iyz="0.0" izz="0.01" />
+        <origin xyz="0.01573 0.0 -0.03029" rpy="0 0 0"/>
+        <mass value="0.19958"/>
+        <inertia
+            ixx="0.000146896"
+            ixy="0.000000005"
+            ixz="0.000001640"
+            iyy="0.000591330"
+            iyz="-0.000000001"
+            izz="0.000653006"/>
       </inertial>
     </link>
@@ -31,7 +37,13 @@
       </visual>
       <inertial>
-        <mass value="1.0" />
-        <origin xyz="0 0 0" rpy="0 0 0" />
-        <inertia ixx="0.01" ixy="0.0" ixz="0.0" iyy="0.01" iyz="0.0" izz="0.01" />
+        <origin xyz="-0.00179 0.00049 -0.15908" rpy="0 0 0"/>
+        <mass value="0.16694"/>
+        <inertia
+            ixx="0.001216063"
+            ixy="0.000000454"
+            ixz="0.000024719"
+            iyy="0.001207669"
+            iyz="-0.000002534"
+            izz="0.000035329"/>
       </inertial>
     </link>
@@ -56,7 +68,13 @@
       </visual>
       <inertial>
-        <mass value="1.0" />
-        <origin xyz="0 0 0" rpy="0 0 0" />
-        <inertia ixx="0.01" ixy="0.0" ixz="0.0" iyy="0.01" iyz="0.0" izz="0.01" />
+        <origin xyz="-0.00179 -0.00050 -0.15908" rpy="0 0 0"/>
+        <mass value="0.16694"/>
+        <inertia
+            ixx="0.001216064"
+            ixy="-0.000000423"
+            ixz="0.000024728"
+            iyy="0.001207666"
+            iyz="0.000002535"
+            izz="0.000035328"/>
       </inertial>
     </link>
@@ -81,7 +99,13 @@
       </visual>
       <inertial>
-        <mass value="1.0" />
-        <origin xyz="0 0 0" rpy="0 0 0" />
-        <inertia ixx="0.01" ixy="0.0" ixz="0.0" iyy="0.01" iyz="0.0" izz="0.01" />
+        <origin xyz="-0.00193 0.0 -0.13250" rpy="0 0 0"/>
+        <mass value="0.15327"/>
+        <inertia
+            ixx="0.001187219"
+            ixy="0.000000002"
+            ixz="0.0"
+            iyy="0.001173746"
+            iyz="0.0"
+            izz="0.000029652"/>
       </inertial>
     </link>
@@ -106,7 +130,13 @@
       </visual>
       <inertial>
-        <mass value="1.0" />
-        <origin xyz="0 0 0" rpy="0 0 0" />
-        <inertia ixx="0.01" ixy="0.0" ixz="0.0" iyy="0.01" iyz="0.0" izz="0.01" />
+        <origin xyz="0.07992 0.0 -0.02000" rpy="0 0 0"/>
+        <mass value="0.20036"/>
+        <inertia
+            ixx="0.000187723"
+            ixy="0.000000002"
+            ixz="-0.000000009"
+            iyy="0.000646427"
+            iyz="-0.000000001"
+            izz="0.000747166"/>
       </inertial>
     </link>
@@ -131,7 +161,13 @@
       </visual>
       <inertial>
-        <mass value="1.0" />
-        <origin xyz="0 0 0" rpy="0 0 0" />
-        <inertia ixx="0.01" ixy="0.0" ixz="0.0" iyy="0.01" iyz="0.0" izz="0.01" />
+        <origin xyz="-0.00179 0.00050 -0.10592" rpy="0 0 0"/>
+        <mass value="0.16694"/>
+        <inertia
+            ixx="0.001216061"
+            ixy="0.000000453"
+            ixz="-0.000024719"
+            iyy="0.001207669"
+            iyz="0.000002625"
+            izz="0.000035328"/>
       </inertial>
     </link>
@@ -160,7 +196,13 @@
       </visual>
       <inertial>
-        <mass value="1.0" />
-        <origin xyz="0 0 0" rpy="0 0 0" />
-        <inertia ixx="0.01" ixy="0.0" ixz="0.0" iyy="0.01" iyz="0.0" izz="0.01" />
+        <origin xyz="-0.00193 0.0 -0.13250" rpy="0 0 0"/>
+        <mass value="0.15327"/>
+        <inertia
+            ixx="0.001187219"
+            ixy="0.000000002"
+            ixz="0.0"
+            iyy="0.001173746"
+            iyz="0.0"
+            izz="0.000029652"/>
       </inertial>
     </link>
@@ -185,7 +227,13 @@
       </visual>
       <inertial>
-        <mass value="1.0" />
-        <origin xyz="0 0 0" rpy="0 0 0" />
-        <inertia ixx="0.01" ixy="0.0" ixz="0.0" iyy="0.01" iyz="0.0" izz="0.01" />
+        <origin xyz="0.08073 0.0 -0.01971" rpy="0 0 0"/>
+        <mass value="0.19958"/>
+        <inertia
+            ixx="0.000146896"
+            ixy="-0.000000005"
+            ixz="-0.000001640"
+            iyy="0.000591330"
+            iyz="-0.000000001"
+            izz="0.000653006"/>
       </inertial>
     </link>
@@ -210,7 +258,13 @@
       </visual>
       <inertial>
-        <mass value="1.0" />
-        <origin xyz="0 0 0" rpy="0 0 0" />
-        <inertia ixx="0.01" ixy="0.0" ixz="0.0" iyy="0.01" iyz="0.0" izz="0.01" />
+        <origin xyz="0.00570 0.00006 -0.02799" rpy="0 0 0"/>
+        <mass value="0.70863"/>
+        <inertia
+            ixx="0.001359548"
+            ixy="0.000003941"
+            ixz="-0.000094799"
+            iyy="0.005895969"
+            iyz="0.000000955"
+            izz="0.006798208"/>
       </inertial>
     </link>
@@ -235,7 +289,13 @@
       </visual>
       <inertial>
-        <mass value="1.0" />
-        <origin xyz="0 0 0" rpy="0 0 0" />
-        <inertia ixx="0.01" ixy="0.0" ixz="0.0" iyy="0.01" iyz="0.0" izz="0.01" />
+        <origin xyz="-0.00179 -0.00049 -0.10592" rpy="0 0 0"/>
+        <mass value="0.16694"/>
+        <inertia
+            ixx="0.001216063"
+            ixy="-0.000000454"
+            ixz="-0.000024719"
+            iyy="0.001207669"
+            iyz="-0.000002534"
+            izz="0.000035329"/>
       </inertial>
     </link>

File: src/alice_xacro_desc/urdf/dn_act_segment.xacro (robot description, xacro)
@@ -19,7 +19,13 @@
       </visual>
       <inertial>
-        <mass value="1.0" />
-        <origin xyz="0 0 0" rpy="0 0 0" />
-        <inertia ixx="0.01" ixy="0.0" ixz="0.0" iyy="0.01" iyz="0.0" izz="0.01" />
+        <origin xyz="0.00042 0.0 -0.00470" rpy="0 0 0"/>
+        <mass value="0.04607"/>
+        <inertia
+            ixx="0.000014850"
+            ixy="0.0"
+            ixz="-0.000000203"
+            iyy="0.000009828"
+            iyz="0.0"
+            izz="0.000013705"/>
       </inertial>
     </link>
@@ -32,7 +38,13 @@
       </visual>
       <inertial>
-        <mass value="1.0" />
-        <origin xyz="0 0 0" rpy="0 0 0" />
-        <inertia ixx="0.01" ixy="0.0" ixz="0.0" iyy="0.01" iyz="0.0" izz="0.01" />
+        <origin xyz="-0.01598 0.00023 -0.07947" rpy="0 0 0"/>
+        <mass value="0.34367"/>
+        <inertia
+            ixx="0.000927312"
+            ixy="-0.000000789"
+            ixz="-0.000065314"
+            iyy="0.001049676"
+            iyz="0.000001769"
+            izz="0.000190178"/>
       </inertial>
     </link>
@@ -58,7 +70,13 @@
       </visual>
       <inertial>
-        <mass value="1.0" />
-        <origin xyz="0 0 0" rpy="0 0 0" />
-        <inertia ixx="0.01" ixy="0.0" ixz="0.0" iyy="0.01" iyz="0.0" izz="0.01" />
+        <origin xyz="0.0 0.0 0.05194" rpy="0 0 0"/>
+        <mass value="0.29579"/>
+        <inertia
+            ixx="0.000366379"
+            ixy="-0.00000000001"
+            ixz="0.0"
+            iyy="0.000366533"
+            iyz="0.00000000001"
+            izz="0.000014856"/>
       </inertial>
     </link>
@@ -89,7 +107,13 @@
       </visual>
       <inertial>
-        <mass value="1.0" />
-        <origin xyz="0 0 0" rpy="0 0 0" />
-        <inertia ixx="0.01" ixy="0.0" ixz="0.0" iyy="0.01" iyz="0.0" izz="0.01" />
+        <origin xyz="-0.00039 0.0 -0.02349" rpy="0 0 0"/>
+        <mass value="0.07743"/>
+        <inertia
+            ixx="0.000026847"
+            ixy="-0.00000000048"
+            ixz="0.000000217"
+            iyy="0.000055486"
+            iyz="0.00000000002"
+            izz="0.000055266"/>
       </inertial>
     </link>

File: src/alice_xacro_desc/urdf/head.xacro (robot description, xacro)
@@ -18,7 +18,13 @@
       </visual>
       <inertial>
-        <mass value="1.0" />
-        <origin xyz="0 0 0" rpy="0 0 0" />
-        <inertia ixx="0.01" ixy="0.0" ixz="0.0" iyy="0.01" iyz="0.0" izz="0.01" />
+        <origin xyz="0.0 -0.00358 0.03195" rpy="0 0 0"/>
+        <mass value="0.05815"/>
+        <inertia
+            ixx="0.000023285"
+            ixy="0.000000000"
+            ixz="-0.000000074"
+            iyy="0.000015710"
+            iyz="-0.000001654"
+            izz="0.000012426"/>
       </inertial>
     </link>
@@ -31,7 +37,13 @@
       </visual>
       <inertial>
-        <mass value="1.0" />
-        <origin xyz="0 0 0" rpy="0 0 0" />
-        <inertia ixx="0.01" ixy="0.0" ixz="0.0" iyy="0.01" iyz="0.0" izz="0.01" />
+        <origin xyz="-0.00377 0.02101 0.03408" rpy="0 0 0"/>
+        <mass value="0.02883"/>
+        <inertia
+            ixx="0.000024978"
+            ixy="0.000000460"
+            ixz="-0.000000341"
+            iyy="0.000008037"
+            iyz="0.000001562"
+            izz="0.000020981"/>
       </inertial>
     </link>

File: src/alice_xacro_desc/urdf/robot.urdf.xacro (robot description, xacro)
@@ -24,7 +24,13 @@
     </visual>
     <inertial>
-      <mass value="1.0" />
-      <origin xyz="0 0 0" rpy="0 0 0" />
-      <inertia ixx="0.01" ixy="0.0" ixz="0.0" iyy="0.01" iyz="0.0" izz="0.01" />
+      <origin xyz="0.01993 0.01512 0.01352" rpy="0 0 0"/>
+      <mass value="9.15148"/>
+      <inertia
+          ixx="0.380681653"
+          ixy="-0.003081798"
+          ixz="0.045436723"
+          iyy="0.247471053"
+          iyz="0.013902336"
+          izz="0.266646562"/>
     </inertial>
   </link>

File: src/alice_xacro_desc/urdf/up_act_segment.xacro (robot description, xacro)
@@ -19,7 +19,13 @@
       </visual>
       <inertial>
-        <mass value="1.0" />
-        <origin xyz="0 0 0" rpy="0 0 0" />
-        <inertia ixx="0.01" ixy="0.0" ixz="0.0" iyy="0.01" iyz="0.0" izz="0.01" />
+        <origin xyz="0.0 0.0 -0.01063" rpy="0 0 0"/>
+        <mass value="0.03745"/>
+        <inertia
+            ixx="0.000012617"
+            ixy="0.0"
+            ixz="0.0"
+            iyy="0.000007833"
+            iyz="0.0"
+            izz="0.000010904"/>
       </inertial>
     </link>
@@ -32,7 +38,13 @@
       </visual>
       <inertial>
-        <mass value="1.0" />
-        <origin xyz="0 0 0" rpy="0 0 0" />
-        <inertia ixx="0.01" ixy="0.0" ixz="0.0" iyy="0.01" iyz="0.0" izz="0.01" />
+        <origin xyz="0.0 0.0 -0.05194" rpy="0 0 0"/>
+        <mass value="0.29579"/>
+        <inertia
+            ixx="0.000366379"
+            ixy="0.00000000001"
+            ixz="0.0"
+            iyy="0.000366533"
+            iyz="0.00000000001"
+            izz="0.000014856"/>
       </inertial>
     </link>
@@ -58,7 +70,13 @@
       </visual>
       <inertial>
-        <mass value="1.0" />
-        <origin xyz="0 0 0" rpy="0 0 0" />
-        <inertia ixx="0.01" ixy="0.0" ixz="0.0" iyy="0.01" iyz="0.0" izz="0.01" />
+        <origin xyz="0.0 0.0 -0.05194" rpy="0 0 0"/>
+        <mass value="0.29579"/>
+        <inertia
+            ixx="0.000366379"
+            ixy="0.00000000001"
+            ixz="0.0"
+            iyy="0.000366533"
+            iyz="0.00000000001"
+            izz="0.000014856"/>
       </inertial>
     </link>
@@ -89,7 +107,13 @@
       </visual>
       <inertial>
-        <mass value="1.0" />
-        <origin xyz="0 0 0" rpy="0 0 0" />
-        <inertia ixx="0.01" ixy="0.0" ixz="0.0" iyy="0.01" iyz="0.0" izz="0.01" />
+        <origin xyz="0.00842 0.0 -0.01380" rpy="0 0 0"/>
+        <mass value="0.04607"/>
+        <inertia
+            ixx="0.000014850"
+            ixy="0.0"
+            ixz="0.000000203"
+            iyy="0.000009828"
+            iyz="0.0"
+            izz="0.000013705"/>
       </inertial>
     </link>
